File: Hardware/FireflyRevB.brd (EAGLE design)
At the start: 101.6 x 82.4 mm, 29 parts, among them IC1 OP-AMP

Commit message: Added the Micro USB and Diodes to the board
Parts:
- removed U$1: USB.MICRO.PWR-BIGGERPADS, CalvEngIO-Connectors:USB-MICRO-01.BIGGERPADS.PWR
- added USB: USB.MICRO.PWR-BIGGERPADS, CalvEngIO-Connectors:USB-MICRO-01.BIGGERPADS.PWR
- C1, C2: device CalvEngIO-Passives:C0402 -> CalvEngIO-Passives:C0603
- moved D1 86.1 mm to (54.6, 34.3), flipped to the bottom
- moved D2 75.5 mm to (36.8, 34.3), flipped to the bottom, turned to 180 degrees
Connections:
- net GND: now also USB.5; no longer U$1.5
- net N$11: now also USB.1; no longer U$1.1
Routing:
- net N$1: track 0.00 -> 22.1 mm
- net N$11: track 0.00 -> 15.8 mm
- net N$9: track 0.00 -> 11.5 mm
Changed lines of the file:
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@@
 <?xml version="1.0" encoding="utf-8"?>
 <!DOCTYPE eagle SYSTEM "eagle.dtd">
-<eagle version="9.1.2">
+<eagle version="9.0.1">
 <drawing>
 <settings>
@@
 <param name="checkStop" value="0"/>
 <param name="checkValues" value="0"/>
-<param name="checkNames" value="1"/>
-<param name="checkWireStubs" value="1"/>
-<param name="checkPolygonWidth" value="0"/>
 <param name="useDiameter" value="13"/>
 <param name="maxErrors" value="50"/>
@@
 <attribute name="NAME" x="34.925" y="40.005" size="1.27" layer="25" rot="R180"/>
 </element>
-<element name="C1" library="CalvEngIO-Passives" package="C0402" value="100n" x="37.465" y="34.925" smashed="yes">
+<element name="C1" library="CalvEngIO-Passives" package="C0603" value="100n" x="37.465" y="34.925" smashed="yes">
 <attribute name="NAME" x="36.322" y="32.639" size="1.27" layer="25"/>
 </element>
@@
 <attribute name="NAME" x="43.815" y="45.339" size="1.27" layer="25" rot="R180"/>
 </element>
-<element name="C2" library="CalvEngIO-Passives" package="C0402" value="100n" x="40.386" y="40.894" smashed="yes" rot="R90">
+<element name="C2" library="CalvEngIO-Passives" package="C0603" value="100n" x="40.386" y="40.894" smashed="yes" rot="R90">
 <attribute name="NAME" x="39.624" y="39.751" size="1.27" layer="25" rot="R90"/>
 </element>
@@
 <element name="U$5" library="CalvEngIO-Logos" package="LINNES.LAB.LOGO" value="LINNES.LAB.LOGO" x="43.18" y="49.53"/>
 <element name="LOGO1" library="CalvEngIO-Logos" package="OSHW-LOGO-L_COPPER" value="OSHW-LOGOL-COPPER" x="36.83" y="48.26"/>
-<element name="U$1" library="CalvEngIO-Connectors" package="USB-MICRO-01.BIGGERPADS.PWR" value="USB.MICRO.PWR-BIGGERPADS" x="-5.08" y="-17.78"/>
-<element name="D1" library="CalvEngIO-DiscreteSemi" package="USC" value="" x="-13.97" y="-17.78"/>
-<element name="D2" library="CalvEngIO-DiscreteSemi" package="USC" value="" x="-17.78" y="-17.78"/>
+<element name="USB" library="CalvEngIO-Connectors" package="USB-MICRO-01.BIGGERPADS.PWR" value="USB.MICRO.PWR-BIGGERPADS" x="22.86" y="26.162" smashed="yes" rot="MR329.1">
+<attribute name="NAME" x="21.453440625" y="31.352196875" size="1.27" layer="26" rot="MR329.1"/>
+</element>
+<element name="D1" library="CalvEngIO-DiscreteSemi" package="USC" value="" x="54.61" y="34.29" smashed="yes" rot="MR0">
+<attribute name="NAME" x="54.61" y="35.39" size="1.27" layer="26" rot="MR0"/>
+<attribute name="VALUE" x="55.88" y="32.625" size="0.635" layer="28" rot="MR0"/>
+</element>
+<element name="D2" library="CalvEngIO-DiscreteSemi" package="USC" value="" x="36.83" y="34.29" smashed="yes" rot="MR180">
+<attribute name="NAME" x="35.56" y="33.19" size="1.27" layer="26" rot="MR180"/>
+<attribute name="VALUE" x="35.56" y="35.955" size="0.635" layer="28" rot="MR180"/>
+</element>
 </elements>
 <signals>
@@
 </polygon>
 <via x="34.29" y="36.83" extent="1-16" drill="0.3048"/>
-<wire x1="40.38" y1="34.925" x2="38.115" y2="34.925" width="0.2032" layer="1"/>
-<wire x1="38.115" y1="34.925" x2="36.21" y2="36.83" width="0.2032" layer="1"/>
+<wire x1="40.38" y1="34.925" x2="38.315" y2="34.925" width="0.2032" layer="1"/>
+<wire x1="38.315" y1="34.925" x2="36.21" y2="36.83" width="0.2032" layer="1"/>
 <wire x1="36.21" y1="36.83" x2="35.98" y2="36.83" width="0.2032" layer="1"/>
 <wire x1="35.98" y1="36.83" x2="34.29" y2="36.83" width="0.2032" layer="1"/>
@@
 <contactref element="LED12" pad="K"/>
 <contactref element="BATTERY" pad="2"/>
-<contactref element="U$1" pad="5"/>
-<wire x1="44.45" y1="64.77" x2="44.45" y2="77.47" width="0" layer="19" extent="1-1"/>
-<wire x1="43.18" y1="45.72" x2="44.45" y2="64.77" width="0" layer="19" extent="16-16"/>
-<wire x1="40.38" y1="34.925" x2="43.18" y2="45.72" width="0" layer="19" extent="1-16"/>
-<wire x1="44.45" y1="21.59" x2="40.38" y2="34.925" width="0" layer="19" extent="1-1"/>
-<wire x1="50.8" y1="17.78" x2="44.45" y2="21.59" width="0" layer="19" extent="1-1"/>
-<wire x1="38.1" y1="17.78" x2="44.45" y2="21.59" width="0" layer="19" extent="1-1"/>
-<wire x1="44.45" y1="10.16" x2="50.8" y2="17.78" width="0" layer="19" extent="1-1"/>
-<wire x1="17.78" y1="38.1" x2="34.29" y2="36.83" width="0" layer="19" extent="1-1"/>
-<wire x1="26.67" y1="52.07" x2="17.78" y2="38.1" width="0" layer="19" extent="1-1"/>
-<wire x1="2.54" y1="24.13" x2="17.78" y2="38.1" width="0" layer="19" extent="1-1"/>
-<wire x1="63.5" y1="52.07" x2="43.18" y2="45.72" width="0" layer="19" extent="16-16"/>
-<wire x1="72.39" y1="38.1" x2="63.5" y2="52.07" width="0" layer="19" extent="1-1"/>
-<wire x1="87.63" y1="24.13" x2="72.39" y2="38.1" width="0" layer="19" extent="1-1"/>
-<wire x1="-3.78" y1="-15.005" x2="2.54" y2="24.13" width="0" layer="19" extent="1-1"/>
+<contactref element="USB" pad="5"/>
 </signal>
 <signal name="PWR">
@@
 <wire x1="40.38" y1="37.465" x2="40.38" y2="38.735" width="0.2032" layer="1"/>
 <wire x1="40.38" y1="38.735" x2="40.386" y2="38.741" width="0.2032" layer="1"/>
-<wire x1="40.386" y1="38.741" x2="40.386" y2="40.244" width="0.2032" layer="1"/>
-<wire x1="40.386" y1="40.244" x2="41.202" y2="41.06" width="0.2032" layer="1"/>
+<wire x1="40.386" y1="38.741" x2="40.386" y2="40.044" width="0.2032" layer="1"/>
+<wire x1="40.386" y1="40.044" x2="41.202" y2="41.06" width="0.2032" layer="1"/>
 <wire x1="41.202" y1="41.06" x2="42.672" y2="41.06" width="0.2032" layer="1"/>
 </signal>
@@
 <contactref element="R5" pad="1"/>
 <wire x1="45.98" y1="36.2057875" x2="45.98" y2="36.195" width="0.2032" layer="1"/>
-<wire x1="40.386" y1="41.544" x2="41.868" y2="43.026" width="0.2032" layer="1"/>
+<wire x1="40.386" y1="41.744" x2="41.868" y2="43.026" width="0.2032" layer="1"/>
 <wire x1="41.868" y1="43.026" x2="41.868" y2="43.3652125" width="0.2032" layer="1"/>
 <wire x1="41.868" y1="43.3652125" x2="42.0167875" y2="43.514" width="0.2032" layer="1"/>
@@
 <contactref element="SWITCH" pad="2"/>
 <contactref element="D1" pad="-"/>
-<wire x1="-12.82" y1="-17.78" x2="43.18" y2="30.81" width="0" layer="19" extent="1-16"/>
-<wire x1="-16.63" y1="-17.78" x2="-12.82" y2="-17.78" width="0" layer="19" extent="1-1"/>
+<wire x1="53.46" y1="34.29" x2="37.98" y2="34.29" width="0.2032" layer="16"/>
+<wire x1="37.98" y1="34.29" x2="39.7" y2="34.29" width="0.2032" layer="16"/>
+<wire x1="39.7" y1="34.29" x2="43.18" y2="30.81" width="0.2032" layer="16"/>
 </signal>
 <signal name="N$9">
 <contactref element="D1" pad="+"/>
 <contactref element="BATTERY" pad="1"/>
-<wire x1="-15.12" y1="-17.78" x2="55.68" y2="45.72" width="0" layer="19" extent="1-16"/>
+<wire x1="55.68" y1="45.72" x2="55.68" y2="34.37" width="0.2032" layer="16"/>
+<wire x1="55.68" y1="34.37" x2="55.76" y2="34.29" width="0.2032" layer="16"/>
 </signal>
 <signal name="N$11">
 <contactref element="D2" pad="+"/>
-<contactref element="U$1" pad="1"/>
-<wire x1="-6.38" y1="-15.005" x2="-18.93" y2="-17.78" width="0" layer="19" extent="1-1"/>
+<contactref element="USB" pad="1"/>
+<wire x1="22.550409375" y1="29.21073125" x2="22.626696875" y2="29.28701875" width="0.2032" layer="16"/>
+<wire x1="22.626696875" y1="29.28701875" x2="22.626696875" y2="30.20193125" width="0.2032" layer="16"/>
+<wire x1="22.626696875" y1="30.20193125" x2="26.714765625" y2="34.29" width="0.2032" layer="16"/>
+<wire x1="26.714765625" y1="34.29" x2="35.68" y2="34.29" width="0.2032" layer="16"/>
 </signal>
 </signals>
-<mfgpreviewcolors>
-<mfgpreviewcolor name="soldermaskcolor" color="0xC8008000"/>
-<mfgpreviewcolor name="silkscreencolor" color="0xFFFEFEFE"/>
-<mfgpreviewcolor name="backgroundcolor" color="0xFF282828"/>
-<mfgpreviewcolor name="coppercolor" color="0xFFFFBF00"/>
-<mfgpreviewcolor name="substratecolor" color="0xFF786E46"/>
-</mfgpreviewcolors>
 </board>
 </drawing>
