File: Hardware/FireflyRevB.sch (EAGLE design)
At the start: 29 parts, among them IC1 OP-AMP

Commit message: Chagned the capacitors to 0603 packages
Parts:
- C1, C2: device CalvEngIO-Passives:CAPACITOR0402 -> CalvEngIO-Passives:CAPACITOR0603
- renumbered U$1 to USB
Changed lines of the file:
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@@
 <?xml version="1.0" encoding="utf-8"?>
 <!DOCTYPE eagle SYSTEM "eagle.dtd">
-<eagle version="9.1.2">
+<eagle version="9.0.1">
 <drawing>
 <settings>
@@
 <part name="IC1" library="SparkFun-IC-Amplifiers" deviceset="OPAMP-DUAL" device="U" value="OP-AMP"/>
 <part name="R1" library="CalvEngIO-Passives" deviceset="RESISTOR" device="0603" value="10k"/>
-<part name="C1" library="CalvEngIO-Passives" deviceset="CAPACITOR" device="0402" value="100n"/>
+<part name="C1" library="CalvEngIO-Passives" deviceset="CAPACITOR" device="0603" value="100n"/>
 <part name="GND1" library="CalvEngIO-Symbols" deviceset="GND" device=""/>
 <part name="R2" library="CalvEngIO-Passives" deviceset="RESISTOR" device="0603" value="10k"/>
 <part name="R3" library="CalvEngIO-Passives" deviceset="RESISTOR" device="0603" value="10k"/>
 <part name="GND3" library="CalvEngIO-Symbols" deviceset="GND" device=""/>
-<part name="C2" library="CalvEngIO-Passives" deviceset="CAPACITOR" device="0402" value="100n"/>
+<part name="C2" library="CalvEngIO-Passives" deviceset="CAPACITOR" device="0603" value="100n"/>
 <part name="R4" library="CalvEngIO-Passives" deviceset="RESISTOR" device="0603" value="10k"/>
 <part name="R5" library="CalvEngIO-Passives" deviceset="RESISTOR" device="0603" value="3.3M"/>
@@
 <part name="U$5" library="CalvEngIO-Logos" deviceset="LINNES.LAB.LOGO" device=""/>
 <part name="LOGO1" library="CalvEngIO-Logos" deviceset="OSHW-LOGO" device="L-COPPER"/>
-<part name="U$1" library="CalvEngIO-Connectors" deviceset="USB.MICRO.PWR" device="-BIGGERPADS"/>
+<part name="USB" library="CalvEngIO-Connectors" deviceset="USB.MICRO.PWR" device="-BIGGERPADS"/>
 <part name="D1" library="CalvEngIO-DiscreteSemi" deviceset="SCHOTTKY" device="-USC"/>
 <part name="D2" library="CalvEngIO-DiscreteSemi" deviceset="SCHOTTKY" device="-USC"/>
@@
 <instance part="R1" gate="G$1" x="50.8" y="86.36" rot="R90"/>
 <instance part="C1" gate="G$1" x="83.82" y="134.62" rot="R90"/>
-<instance part="GND1" gate="1" x="104.14" y="134.62" rot="R90"/>
+<instance part="GND1" gate="1" x="104.14" y="132.08"/>
 <instance part="R2" gate="G$1" x="50.8" y="60.96" rot="R90"/>
 <instance part="R3" gate="G$1" x="101.6" y="73.66" rot="R90"/>
@@
 <instance part="U$5" gate="G$1" x="-7.62" y="63.5"/>
 <instance part="LOGO1" gate="G$1" x="12.7" y="66.04"/>
-<instance part="U$1" gate="G$1" x="5.08" y="101.6"/>
+<instance part="USB" gate="G$1" x="5.08" y="101.6"/>
 <instance part="D1" gate="G$1" x="20.32" y="134.62"/>
 <instance part="D2" gate="G$1" x="17.78" y="106.68"/>
@@
 <pinref part="C1" gate="G$1" pin="2"/>
 <pinref part="GND1" gate="1" pin="GND"/>
-<wire x1="86.36" y1="134.62" x2="101.6" y2="134.62" width="0.1524" layer="91"/>
+<wire x1="86.36" y1="134.62" x2="104.14" y2="134.62" width="0.1524" layer="91"/>
 </segment>
 <segment>
@@
 </segment>
 <segment>
-<pinref part="U$1" gate="G$1" pin="GND"/>
+<pinref part="USB" gate="G$1" pin="GND"/>
 <wire x1="12.7" y1="96.52" x2="15.24" y2="96.52" width="0.1524" layer="91"/>
 <pinref part="GND6" gate="1" pin="GND"/>
@@
 <segment>
 <pinref part="D2" gate="G$1" pin="A"/>
-<pinref part="U$1" gate="G$1" pin="V+"/>
+<pinref part="USB" gate="G$1" pin="V+"/>
 <wire x1="15.24" y1="106.68" x2="12.7" y2="106.68" width="0.1524" layer="91"/>
 </segment>
