File: Hardware/Firefly.brd (EAGLE design)
At the start: 101.6 x 82.4 mm, 29 parts, among them IC1 OP-AMP

Commit message: updates
Parts:
- C1, C2: value 100n -> 2.2u
- LOGO1: value OSHW-LOGOL-COPPER -> OSHW-LOGOL; device CalvEngIO-Logos:OSHW-LOGO-L_COPPER -> CalvEngIO-Logos:OSHW-LOGO-L
- R5: value 3.3M -> 150k
- moved U$5 37.8 mm to (69.4, 22.3), flipped to the bottom
- moved U$4 30.9 mm to (64.8, 24.3), flipped to the bottom
- moved C1 11.0 mm to (46.9, 40.5)
- moved USB 8.10 mm to (15.8, 22.1), turned to 340 degrees
- moved R2 3.58 mm to (38.0, 33.5), turned to 90 degrees
- moved R1 3.22 mm to (37.2, 36.2)
- moved R6 2.10 mm to (51.6, 40.4)
- moved C2 0.81 mm to (40.4, 41.7)
- moved R4 0.36 mm to (50.7, 35.9)
- moved BATTERY 0.23 mm to (43.2, 45.9)
Connections:
- net PWR: now also SWITCH.3; no longer SWITCH.1
Routing:
- net PWR: track 2.23 -> 32.9 mm
- net N$11: track 15.8 -> 25.7 mm
- net GND: track 6.82 -> 0.00 mm, vias 1 -> 0
- net N$1: track 22.1 -> 19.0 mm
- net N$2: track 5.50 -> 4.23 mm
- net N$3: track 208.4 -> 207.7 mm
- added copper zone on layer 1, net GND
- removed copper zone on layer 1, net PWR
Other:
- board text added: "ON"
