File: Hardware/Firefly.sch (EAGLE design)
At the start: 29 parts, among them IC1 OP-AMP

Commit message: updates
Parts:
- C1, C2: value 100n -> 2.2u
- LOGO1: value OSHW-LOGOL-COPPER -> OSHW-LOGOL; device CalvEngIO-Logos:OSHW-LOGOL-COPPER -> CalvEngIO-Logos:OSHW-LOGOL
- R5: value 3.3M -> 150k
Connections:
- net PWR: now also SWITCH.3; no longer SWITCH.1
Other:
- moved on the sheet: LED1
