File: Alternate/Pot-on-Bottom/Firefly-Bottom.brd (EAGLE design)
At the start: 101.6 x 82.2 mm, 26 parts

Commit message: adding everything before organizing...version with potentiometer on top and bottom is complete
Parts:
- removed LOGO1: OSHW-LOGOL, CalvEngIO-Logos:OSHW-LOGO-L
- added R7: 3386F, LinnesLab-Passives:3386F-FOOTPRINT
- moved R5 6.92 mm to (61.3, 39.8)
- moved R6 4.79 mm to (68.7, 33.1)
- moved R4 1.31 mm to (64.1, 32.2)
- moved R3 0.23 mm to (49.3, 39.6)
- moved C2 0.20 mm to (45.6, 39.6)
Connections:
- new net N$8: R5.2, R7.1
- net N$7: now also R7.2; no longer R5.2
Routing:
- net N$7: track 12.7 -> 29.8 mm
- net N$8: track 0.00 -> 16.2 mm
- net N$5: track 24.5 -> 33.0 mm, vias 0 -> 2
- net PWR: track 42.0 -> 38.4 mm
- net N$3: track 214.6 -> 216.4 mm
